Commit message: Change realsense light visualization

File: urdf/_d435.urdf.xacro (robot description, xacro)
@@ -47,6 +47,6 @@
       <origin xyz="${d435_cam_mount_from_center_offset} ${-d435_cam_depth_py} 0" rpy="${M_PI/2} 0 ${M_PI/2}"/>
         <geometry>
-          <!-- <box size="${d435_cam_width} ${d435_cam_height} ${d435_cam_depth}"/> -->
-          <mesh filename="package://realsense2_description/meshes/d435.dae" />
+           <box size="${d435_cam_width} ${d435_cam_height} ${d435_cam_depth}"/>
+          <!--<mesh filename="package://realsense2_description/meshes/d435.dae" /> -->
           <!--<mesh filename="package://realsense2_description/meshes/d435/d435.dae" />-->
         </geometry>
